Commit message: adopt talon urdf from upstream

File: robots/rcta_roman.urdf.xacro (robot description, xacro)
@@ -7,10 +7,10 @@
     <xacro:include filename="$(find roman_model)/gazebo/gazebo.urdf.xacro"/>
     <xacro:talon name="base" namespace="$(arg namespace)"/>
-    <xacro:roman_body name="roman_body" parent="talon" namespace="$(arg namespace)">
+    <xacro:roman_body name="roman_body" parent="base_link" namespace="$(arg namespace)">
         <!--
         <origin xyz="0.27 0 -0.05" rpy="0 1.5708 1.5708"/>
         <origin xyz="0.27 0 0.06" rpy="3.14 1.5708 1.5708"/>
         -->
-        <origin xyz="0.355000 0.000000 0.090000" rpy="3.141592 1.570800 1.570800"/>
+        <origin xyz="0.355000 0.000000 -0.080000" rpy="-1.5708 -1.5708 0.0"/>
     </xacro:roman_body>
     <!-- robosimian_l_arm origin was rpy="0 0.7854 -1.5708?"-->

File: urdf/talon.urdf.xacro (robot description, xacro)
@@ -4,29 +4,17 @@
     <xacro:include filename="$(find roman_model)/control/talon.transmission.xacro"/>
     <xacro:include filename="$(find hector_sensors_description)/urdf/hokuyo_utm30lx.urdf.xacro"/>
+    <xacro:property name="talon_mass" value="100"/>
     <xacro:macro name="talon" params="name namespace">
-        <link name="${name}_footprint"/>
-        <joint name="${name}_footprint_joint" type="fixed">
-            <origin xyz="0 0 0.15203" rpy="0 0 0"/>
-            <parent link="${name}_footprint"/>
-            <child link="${name}_link"/>
-        </joint>
-        <link name="${name}_link"/>
-        <joint name="${name}_joint" type="fixed">
-            <origin xyz="0 0 0" rpy="3.14 0 0"/>
-            <parent link="${name}_link"/>
-            <child link="talon"/>
-        </joint>
-        <link name="talon">
+        <link name="${name}_link">
             <inertial>
-                <mass value="40.0"/>
+                <mass value="${talon_mass}"/>
                 <origin xyz="0 0 0" rpy="0 0 0"/>
-                <!-- NOTE: dummy values for moment of inertia to keep the -->
-                <!-- base from spinning in gazebo -->
-                <inertia ixx="1.0" ixy="0" ixz="0" iyy="1.0" iyz="0" izz="1.0"/>
+                <inertia ixx="6.1754" ixy="0" ixz="0" iyy="10.3160" iyz="0" izz="14.9410"/>
+                <origin xyz="-0.08748 -0.00085 0.09947" />
             </inertial>
             <visual>
-                <origin xyz="0 0 0" rpy="0 0 0"/>
+                <origin xyz="0 0 0" rpy="3.1415926 0 0"/>
                 <geometry>
-<!--                    <box size="0.9 0.6 0.26"/> -->
+                    <!--box size="0.9 0.6 0.26"/-->
                     <mesh filename="package://roman_model/meshes/tl1.stl" scale="1 1 1"/>
                 </geometry>
@@ -37,5 +25,5 @@
             <!-- body -->
             <collision>
-                <origin xyz="0 0 0" rpy="0 0 0"/>
+                <origin xyz="0 0 -0.07" rpy="0 0 0"/>
                 <geometry>
                     <box size="1.070000 0.645000 0.305000"/>
@@ -43,4 +31,5 @@
             </collision>
             <!-- left track -->
+            <!--
             <collision>
                 <origin xyz="0.000000 0.260000 0.000000" rpy="0 0 0"/>
@@ -49,5 +38,7 @@
                 </geometry>
             </collision>
+            -->
             <!-- right track -->
+            <!--
             <collision>
                 <origin xyz="0.000000 -0.260000 0.000000" rpy="0 0 0"/>
@@ -56,7 +47,9 @@
                 </geometry>
             </collision>
+            -->
             <!-- back -->
             <collision>
-                <origin xyz="-0.325000 0.000000 -0.280000" rpy="0 0 0"/>
+                <!--origin xyz="-0.325000 0.000000 0.280000" rpy="0 0 0"/-->
+                <origin xyz="-0.325000 0.000000 0.210000" rpy="0 0 0"/>
                 <geometry>
                     <box size="0.400000 0.645000 0.300000"/>
@@ -67,36 +60,11 @@
             <origin xyz="0.50 0 0.210" rpy="0 0 0"/>
         </xacro:hokuyo_utm30lx_gpu>
-        <joint name="track_left_joint" type="revolute">
-            <origin xyz="0.000000 0.000000 0.000000" rpy="0 0 0"/>
-            <axis xyz="0 0 1"/>
-            <parent link="talon"/>
-            <child link="track_left"/>
-            <limit effort="1000.0" lower="-3.141593" upper="3.141593" velocity="0.5"/>
-            <dynamics damping="0.0" friction="0.0"/>
+        <joint name="${name}_joint" type="fixed">
+            <!--origin xyz="0 0 -0.15" rpy="0 0 0"/-->
+            <origin xyz="0 0 -0.13613" rpy="0 0 0"/>
+            <parent link="${name}_link"/>
+            <child link="${name}_footprint"/>
         </joint>
-        <link name="track_left">
-            <!-- dummy inertial values -->
-            <inertial>
-                <mass value="0.003141"/>
-                <origin xyz="0.000000 0.000000 0.000000" rpy="0 0 0"/>
-                <inertia ixx="0.003141" ixy="0" ixz="0" iyy="0.003141" iyz="0" izz="0.003141"/>
-            </inertial>
-        </link>
-        <joint name="track_right_joint" type="revolute">
-            <origin xyz="0.000000 0.000000 0.000000" rpy="0 0 0"/>
-            <axis xyz="0 0 1"/>
-            <parent link="talon"/>
-            <child link="track_right"/>
-            <limit effort="1000.0" lower="-3.141593" upper="3.141593" velocity="0.5"/>
-            <dynamics damping="0.0" friction="0.0"/>
-        </joint>
-        <link name="track_right">
-            <!-- dummy inertial values -->
-            <inertial>
-                <mass value="0.003141"/>
-                <origin xyz="0.000000 0.000000 0.000000" rpy="0 0 0"/>
-                <inertia ixx="0.003141" ixy="0" ixz="0" iyy="0.003141" iyz="0" izz="0.003141"/>
-            </inertial>
-        </link>
+        <link name="${name}_footprint"/>
         <xacro:talon_gazebo name="${name}" namespace="${namespace}"/>
         <xacro:talon_transmission name="${name}" namespace="${namespace}"/>
