Commit message: offset gripper to match roman1

File: urdf/robosimian_arm.urdf.xacro (robot description, xacro)
@@ -268,5 +268,5 @@
         <!-- attach the robotiq gripper to the arm -->
         <joint name="${prefix}palm_joint" type="fixed">
-            <origin xyz="0.104775 -0.004 0" rpy="3.1415 0 1.57080"/>
+            <origin xyz="0.104775 -0.004 0" rpy="3.1415 -1.57080 1.57080"/>
             <axis xyz="0 0 1"/>
             <parent link="${prefix}link7"/>
