Commit message: add wheels to urdf

File: urdf/talon.urdf.xacro (robot description, xacro)
@@ -4,4 +4,42 @@
     <xacro:include filename="$(find roman_model)/control/talon.transmission.xacro"/>
     <xacro:include filename="$(find hector_sensors_description)/urdf/hokuyo_utm30lx.urdf.xacro"/>
+    <xacro:property name="wheel_mass" value="10"/>
+    <!-- distance between the wheels along x in the base frame -->
+    <xacro:property name="wheelbase" value="0.76"/>
+    <!-- distance between the wheels along y in the base frame -->
+    <xacro:property name="track" value="0.50"/>
+    <!-- vertical offset of the wheels in the base frame -->
+    <xacro:property name="wheel_vertical_offset" value="-0.07"/>
+    <xacro:property name="wheel_length" value="0.154"/>
+    <xacro:property name="wheel_radius" value="0.145"/>
+    <xacro:macro name="roman_wheel" params="wheel_prefix name *origin">
+        <link name="${wheel_prefix}_wheel_link">
+            <collision>
+                <origin xyz="0 0 0" rpy="1.57079 0 0"/>
+                <geometry>
+                    <cylinder length="${wheel_length}" radius="${wheel_radius}"/>
+                </geometry>
+            </collision>
+        </link>
+        <!-- why is this revolute? -->
+        <joint name="${wheel_prefix}_wheel" type="continuous">
+            <parent link="${name}_link"/>
+            <child link="${wheel_prefix}_wheel_link"/>
+            <xacro:insert_block name="origin"/>
+            <axis xyz="0 1 0" rpy="0 0 0"/>
+            <!-- ...with these limits -->
+            <limit effort="1000.0" velocity="9.86"/>
+        </joint>
+        <transmission name="${wheel_prefix}_wheel_trans" type="SimpleTransmission">
+            <type>transmission_interface/SimpleTransmission</type>
+            <actuator name="${wheel_prefix}_wheel_motor">
+                <mechanicalReduction>1</mechanicalReduction>
+            </actuator>
+            <joint name="${wheel_prefix}_wheel">
+                <hardwareInterface>PositionJointInterface</hardwareInterface>
+                <hardwareInterface>VelocityJointInterface</hardwareInterface>
+            </joint>
+        </transmission>
+    </xacro:macro>
     <xacro:property name="talon_mass" value="100"/>
     <xacro:macro name="talon" params="name namespace">
@@ -16,5 +54,4 @@
                 <origin xyz="0 0 0" rpy="3.1415926 0 0"/>
                 <geometry>
-                    <!--box size="0.9 0.6 0.26"/-->
                     <mesh filename="package://roman_model/meshes/tl1.stl" scale="1 1 1"/>
                 </geometry>
@@ -30,25 +67,6 @@
                 </geometry>
             </collision>
-            <!-- left track -->
-            <!--
-            <collision>
-                <origin xyz="0.000000 0.260000 0.000000" rpy="0 0 0"/>
-                <geometry>
-                    <box size="1.070000 0.080000 0.300000"/>
-                </geometry>
-            </collision>
-            -->
-            <!-- right track -->
-            <!--
-            <collision>
-                <origin xyz="0.000000 -0.260000 0.000000" rpy="0 0 0"/>
-                <geometry>
-                    <box size="1.070000 0.080000 0.300000"/>
-                </geometry>
-            </collision>
-            -->
             <!-- back -->
             <collision>
-                <!--origin xyz="-0.325000 0.000000 0.280000" rpy="0 0 0"/-->
                 <origin xyz="-0.325000 0.000000 0.210000" rpy="0 0 0"/>
                 <geometry>
@@ -57,4 +75,16 @@
             </collision>
         </link>
+        <xacro:roman_wheel wheel_prefix="front_left" name="${name}">
+            <origin xyz="${wheelbase/2} ${track/2} ${wheel_vertical_offset}" rpy="0 0 0"/>
+        </xacro:roman_wheel>
+        <xacro:roman_wheel wheel_prefix="front_right" name="${name}">
+            <origin xyz="${wheelbase/2} ${-track/2} ${wheel_vertical_offset}" rpy="0 0 0"/>
+        </xacro:roman_wheel>
+        <xacro:roman_wheel wheel_prefix="rear_left" name="${name}">
+            <origin xyz="${-wheelbase/2} ${track/2} ${wheel_vertical_offset}" rpy="0 0 0"/>
+        </xacro:roman_wheel>
+        <xacro:roman_wheel wheel_prefix="rear_right" name="${name}">
+            <origin xyz="${-wheelbase/2} ${-track/2} ${wheel_vertical_offset}" rpy="0 0 0"/>
+        </xacro:roman_wheel>
         <xacro:hokuyo_utm30lx_gpu name="base_laser" parent="base_link" ros_topic="base_scan" update_rate="20.0" ray_count="1080" min_angle="-130" max_angle="130">
             <origin xyz="0.50 0 0.210" rpy="0 0 0"/>
