Commit message: update some gazebo urdf extensions and configure kinematic sim plugin

File: control/talon.transmission.xacro (robot description, xacro)
@@ -2,20 +2,40 @@
 <robot xmlns:xacro="http://ros.org/wiki/xacro">
     <xacro:macro name="talon_transmission" params="name namespace">
-        <transmission name="track_left_joint_transmission">
+        <transmission name="front_left_wheel_transmission">
             <type>transmission_interface/SimpleTransmission</type>
-            <joint name="track_left_joint">
+            <joint name="front_left_wheel">
                 <hardwareInterface>EffortJointInterface</hardwareInterface>
             </joint>
-            <actuator name="track_left_joint_motor">
+            <actuator name="front_left_wheel_motor">
                 <hardwareInterface>EffortJointInterface</hardwareInterface>
                 <mechanicalReduction>1</mechanicalReduction>
             </actuator>
         </transmission>
-        <transmission name="track_right_joint_transmission">
+        <transmission name="front_right_wheel_transmission">
             <type>transmission_interface/SimpleTransmission</type>
-            <joint name="track_right_joint">
+            <joint name="front_right_wheel">
                 <hardwareInterface>EffortJointInterface</hardwareInterface>
             </joint>
-            <actuator name="track_right_joint_motor">
+            <actuator name="front_right_wheel_motor">
+                <hardwareInterface>EffortJointInterface</hardwareInterface>
+                <mechanicalReduction>1</mechanicalReduction>
+            </actuator>
+        </transmission>
+        <transmission name="rear_left_wheel_transmission">
+            <type>transmission_interface/SimpleTransmission</type>
+            <joint name="rear_left_wheel">
+                <hardwareInterface>EffortJointInterface</hardwareInterface>
+            </joint>
+            <actuator name="rear_left_wheel_motor">
+                <hardwareInterface>EffortJointInterface</hardwareInterface>
+                <mechanicalReduction>1</mechanicalReduction>
+            </actuator>
+        </transmission>
+        <transmission name="rear_right_wheel_transmission">
+            <type>transmission_interface/SimpleTransmission</type>
+            <joint name="rear_right_wheel">
+                <hardwareInterface>EffortJointInterface</hardwareInterface>
+            </joint>
+            <actuator name="rear_right_wheel_motor">
                 <hardwareInterface>EffortJointInterface</hardwareInterface>
                 <mechanicalReduction>1</mechanicalReduction>

File: gazebo/gazebo.urdf.xacro (robot description, xacro)
@@ -7,5 +7,5 @@
                 <robotNamespace>rcta_roman</robotNamespace>
             </xacro:if>
-            <robotSimType>gazebo_ros_control/DefaultRobotHWSim</robotSimType>
+            <robotSimType>roman_simulation/KinematicRobotHWSim</robotSimType>
         </plugin>
     </gazebo>

File: gazebo/talon.gazebo.xacro (robot description, xacro)
@@ -7,4 +7,12 @@
             <minDepth>0.01</minDepth>
         </gazebo>
+        <gazebo reference="front_left_wheel_link"/>
+        <gazebo reference="front_left_wheel"/>
+        <gazebo reference="front_right_wheel_link"/>
+        <gazebo reference="front_right_wheel"/>
+        <gazebo reference="rear_left_wheel_link"/>
+        <gazebo reference="rear_left_wheel"/>
+        <gazebo reference="rear_right_wheel_link"/>
+        <gazebo reference="rear_right_wheel"/>
     </xacro:macro>
 </robot>
